File: hardware/WingBoard/WingBoard.kicad_pcb (KiCad board)
At the start: 2 copper layers, 40 x 90 mm, 103 parts, among them J101 UPDI, J102 UART0, J201 PWR_SEL, J202 Vin, J301 MPU-6050, J302 BN-220 GPS, J303 I2C_X_5V, J304 I2C_X_3.3V, J401 PWM_IN1, J402 PWM_IN2, J403 PWM_IN3, J404 PWM_IN4, J405 PWM_IN5, J406 PWM_IN6, J407 PWM_OUT1, J408 PWM_OUT2, J409 PWM_OUT3, J410 PWM_OUT4, J411 PWM_OUT5, J412 PWM_OUT6, Q301 BSS138, Q302 BSS138, SW101 DIPA, SW102 DIPB, SW103 SW_SPST, SW201 SW_POWER, U101 ATmega4809-A, U201 AZ1117-5.0, U202 AZ1117-3.3, U301 MMC5603, U302 BMP581, U401 PCA9685PW, U402 ATtiny85-20S, U403 74157

Commit message: Hardware layout v0.1 complete.
Parts:
- removed D101: STAT0, LED_SMD:LED_0805_2012Metric_Pad1.15x1.40mm_HandSolder
- removed D102: STAT1, LED_SMD:LED_0805_2012Metric_Pad1.15x1.40mm_HandSolder
- removed D103: STAT2, LED_SMD:LED_0805_2012Metric_Pad1.15x1.40mm_HandSolder
- removed D104: STAT3, LED_SMD:LED_0805_2012Metric_Pad1.15x1.40mm_HandSolder
- removed D202: 3V, LED_SMD:LED_0805_2012Metric_Pad1.15x1.40mm_HandSolder
- removed R104, R105, R106, R107: 1k, Resistor_SMD:R_0805_2012Metric_Pad1.20x1.40mm_HandSolder
- removed R202: LED_PWR, Resistor_SMD:R_0805_2012Metric_Pad1.20x1.40mm_HandSolder
- removed SW102: DIPB, Button_Switch_SMD:SW_DIP_SPSTx02_Slide_Copal_CHS-02B_W7.62mm_P1.27mm
- removed TP101: VDD_TP, TestPoint:TestPoint_Pad_D1.5mm
- removed TP105, TP106: TP_GND, TestPoint:TestPoint_Pad_D1.5mm
- removed TP201: TP_5V, TestPoint:TestPoint_Pad_D1.5mm
- removed TP202: TP_3.3V, TestPoint:TestPoint_Pad_D1.5mm
- removed TP301: TP_SDA_3.3v, TestPoint:TestPoint_Pad_D1.5mm
- removed TP302: TP_SCL_3.3v, TestPoint:TestPoint_Pad_D1.5mm
- C101, C301, C302, JP301: moved to B.Cu
- moved J412 65.1 mm to (141.5, 123.4), turned to -90 degrees
- moved J304 63.1 mm to (169.0, 65.8), turned to 0 degrees
- moved TP102 58.6 mm to (171.2, 58.0)
- moved J411 57.8 mm to (141.5, 119.4), turned to -90 degrees
- moved J303 54.7 mm to (169.0, 71.8), turned to 0 degrees
- moved TP103 53.4 mm to (171.2, 61.6)
- moved JP301 52.1 mm to (161.9, 76.2), turned to 90 degrees
- moved U403 51.8 mm to (147.7, 115.4), turned to -90 degrees
- moved J410 50.7 mm to (141.5, 115.4), turned to -90 degrees
- moved R301 50.0 mm to (162.6, 63.4), turned to 0 degrees
- moved U301 49.2 mm to (161.2, 71.6), turned to 90 degrees
- moved U302 48.8 mm to (159.2, 76.6), turned to 0 degrees
- moved C301 48.4 mm to (156.8, 71.8)
- moved C302 47.5 mm to (156.8, 75.9), turned to -90 degrees
- moved Q301 45.8 mm to (162.6, 66.6), turned to 90 degrees
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Connections:
- net /PWM Connections/PWM CTRL B0 renamed /PWM Connections/PWM TO MUX 1
- net /PWM Connections/PWM CTRL B1 renamed /PWM Connections/PWM TO MUX 2
- net /PWM Connections/PWM CTRL B2 renamed /PWM Connections/PWM TO MUX 3
- net /PWM Connections/PWM CTRL B3 renamed /PWM Connections/PWM TO MUX 4
- net Net-(BT201-Pad1) renamed /Power Assembly/BAT+
- net Net-(C201-Pad1) renamed /Power Assembly/5V_REG_IN
- net Net-(J407-Pad1) renamed /PWM Connections/PWM O1
- net Net-(J408-Pad1) renamed /PWM Connections/PWM O2
- net Net-(J409-Pad1) renamed /PWM Connections/PWM O3
- net Net-(J410-Pad1) renamed /PWM Connections/PWM O4
- C204 pad 1: VDD -> +5VA
- D105 pad 1: Net-(D105-Pad1) -> /STAT_4
- D105 pad 2: VDD -> Net-(D105-Pad2)
- D106 pad 1: Net-(D106-Pad1) -> /STAT_3
- D106 pad 2: VDD -> Net-(D106-Pad2)
- D107 pad 1: Net-(D107-Pad1) -> /STAT_2
- D107 pad 2: VDD -> Net-(D107-Pad2)
- D108 pad 1: Net-(D108-Pad1) -> /STAT_1
- D108 pad 2: VDD -> Net-(D108-Pad2)
- D201 pad 2: VCC -> VDD
- R108 pad 1: Net-(D105-Pad1) -> VDD
- R108 pad 2: Net-(R108-Pad2) -> Net-(D105-Pad2)
- R109 pad 1: Net-(D106-Pad1) -> VDD
- R109 pad 2: Net-(R109-Pad2) -> Net-(D106-Pad2)
- R110 pad 1: Net-(D107-Pad1) -> VDD
- R110 pad 2: Net-(R110-Pad2) -> Net-(D107-Pad2)
- R111 pad 1: Net-(D108-Pad1) -> VDD
- R111 pad 2: Net-(R111-Pad2) -> Net-(D108-Pad2)
- U101 pad 16: unconnected-(U101-Pad16) -> MCU_PWM_OUT_4
- U101 pad 17: unconnected-(U101-Pad17) -> MCU_PWM_OUT_3
- U101 pad 18: unconnected-(U101-Pad18) -> MCU_PWM_OUT_2
- U101 pad 19: unconnected-(U101-Pad19) -> MCU_PWM_OUT_1
- U101 pad 20: Net-(R104-Pad2) -> /STAT_1
- U101 pad 21: Net-(R105-Pad2) -> /STAT_2
- U101 pad 22: Net-(R106-Pad2) -> /STAT_3
- U101 pad 23: Net-(R107-Pad2) -> /STAT_4
- U101 pad 24: Net-(R108-Pad2) -> unconnected-(U101-Pad24)
- U101 pad 25: Net-(R109-Pad2) -> unconnected-(U101-Pad25)
- U101 pad 26: Net-(R110-Pad2) -> unconnected-(U101-Pad26)
- U101 pad 27: Net-(R111-Pad2) -> unconnected-(U101-Pad27)
- U101 pad 30: /DIP_A0 -> unconnected-(U101-Pad30)
- U101 pad 31: /DIP_A1 -> unconnected-(U101-Pad31)
- U101 pad 32: /DIP_B0 -> unconnected-(U101-Pad32)
- U101 pad 33: /DIP_B1 -> unconnected-(U101-Pad33)
- U101 pad 35: unconnected-(U101-Pad35) -> /DIP_A1
- U101 pad 36: MCU_PWM_OUT_1 -> /DIP_A0
- U101 pad 37: MCU_PWM_OUT_2 -> unconnected-(U101-Pad37)
- U101 pad 38: MCU_PWM_OUT_3 -> unconnected-(U101-Pad38)
- U101 pad 39: MCU_PWM_OUT_4 -> unconnected-(U101-Pad39)
- U403 pad 16: VCC -> VDD
Routing:
- net VDD: track 0.00 -> 261.7 mm, vias 0 -> 11
- net GND: track 0.00 -> 145.8 mm, vias 0 -> 16
- net I2C_SCL: track 0.00 -> 103.6 mm, vias 0 -> 1
- net I2C_SDA: track 0.00 -> 102.6 mm, vias 0 -> 4
- net +5VA: track 0.00 -> 92.0 mm
- net PWM_IN_1: track 0.00 -> 75.0 mm, vias 0 -> 4
- net PWM_IN_2: track 0.00 -> 70.7 mm, vias 0 -> 4
- net PWM_IN_3: track 0.00 -> 67.2 mm, vias 0 -> 4
- net PWM_IN_4: track 0.00 -> 64.0 mm, vias 0 -> 2
- net +3V3: track 0.00 -> 47.0 mm, vias 0 -> 5
- net /DIP_A0: track 0.00 -> 42.2 mm
- net /DIP_A1: track 0.00 -> 41.0 mm
- net /PWM Connections/CTRL_OVERRIDE: track 0.00 -> 38.5 mm, vias 0 -> 2
- net MCU_RESET: track 0.00 -> 35.1 mm, vias 0 -> 2
- net UART_1_MCU_RX: track 0.00 -> 34.9 mm, vias 0 -> 2
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- added copper zone on F.Cu, net /Power Assembly/BAT+
- added copper zone on B.Cu, net GND
- added copper zone on F.Cu, net GND
Other:
- board text added: "+"
- board text added: "+ G C D"
- board text added: "-"
- board text added: "0"
- board text added: "1"
- board text added: "2"
- board text added: "2-3s LiPo"
- board text added: "3"
- board text added: "4"
- board text added: "5"
- board text added: "6"
- board text added: "ATmega4809"
- board text added: "ATtiny85"
- board text added: "Bat"
- board text added: "CH1"
- board text added: "CH2"
- board text added: "CH3"
- board text added: "CH4"
- board text added: "G + T R"
- board text added: "GND"
- board text added: "GPS"
- board text added: "Gnd"
- board text added: "I2C-3.3v"
- board text added: "I2C-5v"
- board text added: "IN"
- board text added: "JLCJLCJLCJLC"
- board text added: "MCU I/O"
- board text added: "MMC 5603"
- board text added: "MPU-6050"
- board text added: "OUT"
- board text added: "PWM IC"
- board text added: "Pdwn"
- board text added: "Pup"
- board text added: "Pwr"
- board text added: "Rcvr"
- board text added: "Rx"
- board text added: "SCL"
- board text added: "SDA"
- board text added: "Sig"
- board text added: "Status"
- board text added: "Tx"
- board text added: "UPDI"
- board text added: "Vdd"
- board text added: "Wingboard Ver: 0.1"

Commit message: Final wingboard v0.1 hardware design.
Parts:
- U302: value BMP581 -> BMP 581
- U402: value ATtiny85-20S -> ATtiny85
Routing:
- net VDD: track 261.7 -> 277.0 mm, vias 11 -> 12
- net +3V3: track 47.0 -> 58.1 mm, vias 5 -> 6
- net GND: track 145.8 -> 150.3 mm, vias 16 -> 17
- net UART_1_MCU_TX: track 34.7 -> 34.1 mm
Other:
- board text added: "09-21-2022"
- board text added: "100n"
- board text added: "10k"
- board text added: "10u"
- board text added: "1K"
- board text added: "220"
- board text added: "2u2"
- board text added: "5V In"
- board text added: "ATmega 4809"
- board text added: "AZ1117-3.3v"
- board text added: "AZ1117-5v"
- board text added: "Ben Emmett"
- board text added: "CSB"
- board text added: "D"
- board text added: "G + R T"
- board text added: "PCA9685 PWM IC"
- board text added: "Power Select"
- board text added: "SCL Pup"
- board text added: "SDA Pup"
- board text added: "SN74157 Mux"
- board text removed: "ATmega4809"
- board text removed: "G + T R"
